File: V2.0/BicycLED_POV.sch (KiCad schematic (older format))
At the start: 65 parts, among them IC1 AT45DBXX1, IC2 AT91SAM7S512/256/128/64/321-AU, J1 CONN_USB, J2 CONN_MICRO_SD, P1 CONN_2, Q1 NTR417P, Q2 NTR417P, Q3 2N2002K, SW1 bootloader, U1 CONN_JTAG_ARM, U3 MCP73811/2, U4 AH173, U5 FAN2502-XX, X1 18.432 MHz

Commit message: 
Connections:
- net labels removed: JTAG_CLK
Changed lines of the file:
@@
-EESchema Schematic File Version 2  date 29/05/2010 05:31:03
+EESchema Schematic File Version 2  date 03/06/2010 20:35:50
 LIBS:regul
 LIBS:switch_FSM2JSMA
@@
 Sheet 1 2
 Title "   BicycLED POV"
-Date "29 may 2010"
+Date "3 jun 2010"
 Rev "v 2.0"
 Comp "Hardware BOX                                http://code.google.com/p/bicycleledpov"
@@
 JTAG_TMS
 Text GLabel 2900 5100 2    55   Input ~ 0
-JTAG_CLK
+JTAG_TCK
 Text GLabel 2900 5300 2    55   Input ~ 0
 JTAG_TDO
